Commit message: added collisions

File: URDFtests/src/robot_descr/urdf/description.urdf (robot description, URDF)
Before this commit: robot myfirst, 15 links, 14 joints
Links:
- link drone_base: geometry collision cylinder length=0.05 radius=0.3; visual cylinder length=0.05 radius=0.3
- link drone_lding_gear_L: geometry collision cylinder length=0.6 radius=0.03; visual cylinder length=0.6 radius=0.03
- link drone_lding_gear_R: geometry collision cylinder length=0.6 radius=0.03; visual cylinder length=0.6 radius=0.03
- link drone_leg_link_LL: geometry collision cylinder length=0.4 radius=0.02; visual cylinder length=0.4 radius=0.02
- link drone_leg_link_LR: geometry collision cylinder length=0.4 radius=0.02; visual cylinder length=0.4 radius=0.02
- link drone_leg_link_RL: geometry collision cylinder length=0.4 radius=0.02; visual cylinder length=0.4 radius=0.02
- link drone_leg_link_RR: geometry collision cylinder length=0.4 radius=0.02; visual cylinder length=0.4 radius=0.02
- link prop_LL: geometry collision box size=0.002 0.02 0.5; visual box size=0.002 0.02 0.5
- link prop_LR: geometry collision box size=0.002 0.02 0.5; visual box size=0.002 0.02 0.5
- link prop_RL: geometry collision box size=0.002 0.02 0.5; visual box size=0.002 0.02 0.5
- link prop_RR: geometry collision box size=0.002 0.02 0.5; visual box size=0.002 0.02 0.5
- link prop_handle_LL: geometry collision cylinder length=0.6 radius=0.03; visual cylinder length=0.6 radius=0.03
- link prop_handle_LR: geometry collision cylinder length=0.6 radius=0.03; visual cylinder length=0.6 radius=0.03
- link prop_handle_RL: geometry collision cylinder length=0.6 radius=0.03; visual cylinder length=0.6 radius=0.03
- link prop_handle_RR: geometry collision cylinder length=0.6 radius=0.03; visual cylinder length=0.6 radius=0.03
